File: board.sch (KiCad schematic (older format))
At the start: 18 parts, among them P1 CONN_8, P2 CONN_8, U1 74LS595, U2 74LS595, U3 CD74ACT257M96, U4 CD74ACT257M96, U5 74HC04, U6 FDC6305N, U7 RG7SEG

Commit message: Update schematic, initial board layout, add gerber files output for easier board creation
Parts:
- removed U5: 74HC04, ~, symbol 74HC04
- added U5: 74LVC1G14, ~, symbol 74LVC1G14
- R1: value R -> 150
Connections:
- net labels added: Clk, Din, Dout, Glatch, OE, R/G sel, Rlatch
- wire segments 197 -> 199
Changed lines of the file:
@@
 LIBS:contrib
 LIBS:valves
-LIBS:RG7seg
 LIBS:NL37WZ14
 LIBS:CD74ACT257M96
@@
 Sheet 1 1
 Title ""
-Date "28 may 2014"
+Date "9 jun 2014"
 Rev ""
 Comp ""
@@
 P 10200 5700
 F 0 "R1" V 10280 5700 50  0000 C CNN
-F 1 "R" V 10200 5700 50  0000 C CNN
+F 1 "150" V 10200 5700 50  0000 C CNN
 F 2 "" H 10200 5700 60  0001 C CNN
 F 3 "" H 10200 5700 60  0001 C CNN
@@
 $EndComp
 $Comp
-L GND #PWR7
+L GND #PWR01
 U 1 1 51B3AF80
 P 8200 5550
-F 0 "#PWR7" H 8200 5550 30  0001 C CNN
+F 0 "#PWR01" H 8200 5550 30  0001 C CNN
 F 1 "GND" H 8200 5480 30  0001 C CNN
 F 2 "" H 8200 5550 60  0001 C CNN
@@
 $EndComp
 $Comp
-L GND #PWR5
+L GND #PWR02
 U 1 1 5383FC6E
 P 4550 6600
-F 0 "#PWR5" H 4550 6600 30  0001 C CNN
+F 0 "#PWR02" H 4550 6600 30  0001 C CNN
 F 1 "GND" H 4550 6530 30  0001 C CNN
 F 2 "" H 4550 6600 60  0000 C CNN
@@
 $EndComp
 $Comp
-L VCC #PWR6
+L VCC #PWR03
 U 1 1 5383FD8A
 P 6350 1700
-F 0 "#PWR6" H 6350 1800 30  0001 C CNN
+F 0 "#PWR03" H 6350 1800 30  0001 C CNN
 F 1 "VCC" H 6350 1800 30  0000 C CNN
 F 2 "" H 6350 1700 60  0000 C CNN
@@
 $EndComp
 $Comp
-L 74HC04 U5
-U 1 1 53840210
-P 7250 5900
-F 0 "U5" H 7400 6000 40  0000 C CNN
-F 1 "74HC04" H 7450 5800 40  0000 C CNN
-F 2 "~" H 7250 5900 60  0000 C CNN
-F 3 "~" H 7250 5900 60  0000 C CNN
-	1    7250 5900
-	1    0    0    -1
-$EndComp
-$Comp
 L RG7SEG U7
 U 1 1 517B3464
@@
 F 3 "" H 600 2100 60  0000 C CNN
 	1    600  2100
-	-1   0    0    -1
+	-1   0    0    1
 $EndComp
 $Comp
@@
 F 3 "" H 600 3300 60  0000 C CNN
 	1    600  3300
-	-1   0    0    -1
-$EndComp
-$Comp
-L VCC #PWR3
+	-1   0    0    1
+$EndComp
+$Comp
+L VCC #PWR04
 U 1 1 538422C3
 P 1350 1450
-F 0 "#PWR3" H 1350 1550 30  0001 C CNN
+F 0 "#PWR04" H 1350 1550 30  0001 C CNN
 F 1 "VCC" H 1350 1550 30  0000 C CNN
 F 2 "" H 1350 1450 60  0000 C CNN
@@
 $EndComp
 $Comp
-L GND #PWR2
+L GND #PWR05
 U 1 1 538422D2
 P 1250 5400
-F 0 "#PWR2" H 1250 5400 30  0001 C CNN
+F 0 "#PWR05" H 1250 5400 30  0001 C CNN
 F 1 "GND" H 1250 5330 30  0001 C CNN
 F 2 "" H 1250 5400 60  0000 C CNN
@@
 $EndComp
 $Comp
-L GND #PWR4
+L GND #PWR06
 U 1 1 53852E58
 P 3100 7450
-F 0 "#PWR4" H 3100 7450 30  0001 C CNN
+F 0 "#PWR06" H 3100 7450 30  0001 C CNN
 F 1 "GND" H 3100 7380 30  0001 C CNN
 F 2 "" H 3100 7450 60  0000 C CNN
@@
 $EndComp
 $Comp
-L VCC #PWR1
+L VCC #PWR07
 U 1 1 53852E67
 P 1100 6300
-F 0 "#PWR1" H 1100 6400 30  0001 C CNN
+F 0 "#PWR07" H 1100 6400 30  0001 C CNN
 F 1 "VCC" H 1100 6400 30  0000 C CNN
 F 2 "" H 1100 6300 60  0000 C CNN
@@
 	8600 4200 8900 4200
 Wire Wire Line
-	8600 4300 8900 4300
-Wire Wire Line
 	10450 4200 10450 5700
 Wire Wire Line
@@
 Wire Wire Line
 	6650 4200 8200 4200
-Wire Wire Line
-	8200 4300 6750 4300
-Wire Wire Line
-	6750 4300 6750 5600
 Wire Wire Line
 	6750 5600 4250 5600
@@
 Wire Wire Line
 	8800 5050 8800 4000
+$Comp
+L 74LVC1G14 U5
+U 1 1 538E7F08
+P 7250 5900
+F 0 "U5" H 7400 6000 40  0000 C CNN
+F 1 "74LVC1G14" H 7450 5800 40  0000 C CNN
+F 2 "~" H 7250 5900 60  0000 C CNN
+F 3 "~" H 7250 5900 60  0000 C CNN
+	1    7250 5900
+	1    0    0    -1
+$EndComp
+Wire Wire Line
+	8600 4400 8700 4400
+Wire Wire Line
+	8700 4400 8700 4300
+Wire Wire Line
+	8700 4300 8900 4300
+Wire Wire Line
+	6750 4400 6750 5600
+Wire Wire Line
+	6750 4400 8200 4400
+Text Label 1450 1850 0    60   ~ 0
+Din
+Text Label 2900 3700 0    60   ~ 0
+Dout
+Text Label 1000 1950 0    60   ~ 0
+Clk
+Text Label 1050 2050 0    60   ~ 0
+Rlatch
+Text Label 1100 2150 0    60   ~ 0
+Glatch
+Text Label 1150 2250 0    60   ~ 0
+R/G sel
+Text Label 1200 2350 0    60   ~ 0
+OE
 $EndSCHEMATC
